Commit message: Fix wheel visual alignment
Co-authored-by: Copilot <223556219+Copilot@users.noreply.github.com>

File: urdf/rover.urdf.xacro (robot description, xacro)
@@ -57,5 +57,5 @@
     </inertial>
     <visual>
-      <origin xyz="-0.202496 0.121044 0.0070156" rpy="1.5708 0 0" />
+      <origin xyz="-0.202496 -0.013323  -0.140697" rpy="1.5708 0 0" />
       <geometry>
         <mesh filename="${mesh_dir}/fore_right_wheel_0_Body1.stl" scale="0.001 0.001 0.001" />
@@ -77,5 +77,5 @@
     </inertial>
     <visual>
-      <origin xyz="-0.00155815 0.0753456 -0.0227239" rpy="1.5708 0 0" />
+      <origin xyz="-0.001558 -0.043074 -0.094972" rpy="1.5708 0 0" />
       <geometry>
         <mesh filename="${mesh_dir}/back_right_wheel_0_Body1.stl" scale="0.001 0.001 0.001" />
@@ -97,5 +97,5 @@
     </inertial>
     <visual>
-      <origin xyz="-0.227255 -0.0313744 -0.0344146" rpy="1.5708 0 0" />
+      <origin xyz="-0.227255 -0.014410 0.051350" rpy="1.5708 0 0" />
       <geometry>
         <mesh filename="${mesh_dir}/Component87_0_Body1.stl" scale="0.001 0.001 0.001" />
@@ -117,5 +117,5 @@
     </inertial>
     <visual>
-      <origin xyz="-0.000613365 0.0399906 -1.39496e-05" rpy="1.5708 0 0" />
+      <origin xyz="-0.000613 0.019990 -0.020014" rpy="1.5708 0 0" />
       <geometry>
         <mesh filename="${mesh_dir}/back_left_wheel_0_Body1.stl" scale="0.001 0.001 0.001" />
